Commit message: Update .gitignore to exclude database environment file and modify TurtleBot3ManualConfig.urdf joint orientation

File: Nav2SLAMExampleProject/Assets/turtlebot3/TurtleBot3ManualConfig.urdf (robot description, URDF)
Before this commit: robot TurtleBot3ManualConfig, 7 links, 6 joints
Joints:
- joint pump_hose_joint: origin xyz=0.1 0 0.1 rpy=0 0 0 -> xyz=0.1 0 0.1 rpy=1.57 0 0

Commit message: ROS2 Python and Unity C# code in WSL. Hopefully appears on Github and opens in Unity

File: Nav2SLAMExampleProject/Assets/turtlebot3/TurtleBot3ManualConfig.urdf (robot description, URDF)
Before this commit: robot TurtleBot3ManualConfig, 7 links, 6 joints
Joints:
- joint pump_hose_joint: origin xyz=0.1 0 0.1 rpy=1.57 0 0 -> xyz=0.1 0 0.1 rpy=0 0 0
